File: hardware/v0.1a/SAMR34.sch (KiCad schematic (older format))
At the start: 53 parts, among them U1 SKY13373, U8 ATSAMR34J18B, U9 PE4259

Commit message: Fixing up some errors after shuffle of libraries.
Parts:
- removed ANT1, ANT?1: 433Mhz CHIP, symbol gpsLogger:ANT
- added A? (x2): pkl_ANTENNA, symbol pkl_misc:pkl_ANTENNA
- added C? (x4): 100nF, Capacitors_SMD:C_0402_NoSilk, symbol device:C_Small
- U1: symbol gpsLogger:SKY13373 -> gkl_rf:SKY13373
- U8: symbol gpsLogger:ATSAMR34J18B -> gkl_microchip:ATSAMR34J18B
- U9: symbol gpsLogger:PE4259 -> gkl_rf:PE4259
Connections:
- net labels added: +3V3, AVDD
- net labels removed: VDDA
- wire segments 206 -> 238

Commit message: Changed USB connector. Updated board outline. Updates to footprints to use 3d models. Add FLASH memory.
Parts:
- removed C30, C32: 18pF, Capacitors_SMD:C_0402_NoSilk, symbol device:C_Small
- removed U9: PE4259, TO_SOT_Packages_SMD:SOT-363_SC-70-6, symbol gkl_rf:PE4259
- added L18: 1k, pkl_dipol:L_0402, symbol device:Ferrite_Bead_Small
- added U4: SKY13373, gkl_housings_qfn:QFN-12-1EP_3x3mm_P0.5mm_EP1.65x1.65mm, symbol gkl_rf:SKY13373
- A1: renamed from A?; footprint (none) -> gkl_antenna:0900AT43A0070 - 900MHz Wide band ISM Chip Antenna
- A2: renamed from A?; footprint (none) -> gkl_antenna:0433AT62A0020 - 433MHz 25x5x1mm chip antenna
- C1, C2, C3, C6: renamed from C?; footprint Capacitors_SMD:C_0402_NoSilk -> pkl_dipol:C_0402
- C10, C12, C13, C18, C19, C20, C21, C22, C23, C24, C25, C26, C27, C28, C29, C31, C33, C34, C35, C36, C37, C38, C39, C4, C40, C41, C42, C5, C7, C8: footprint Capacitors_SMD:C_0402_NoSilk -> pkl_dipol:C_0402
- L1, L10, L11, L12, L13, L14, L15, L16, L2, L3, L4, L5, L6, L7, L8, L9: footprint Inductors_SMD:L_0402 -> pkl_dipol:L_0402
- U1: footprint (none) -> gkl_housings_qfn:QFN-12-1EP_3x3mm_P0.5mm_EP1.65x1.65mm
- U8: footprint (none) -> gkl_housings_bga:TFBGA-64_6.0x6.0mm_Layout8x8_P0.65mm
Connections:
- net labels added: SHDN
- wire segments 238 -> 251
- no-connect marks 0 -> 3
Other:
- note added: "SHDN (V1=0, V2=0)\nRFC = J1 (V1=0, V2=1)\nRFC = J2 (V1=1, V2=0)\nRFC = J3 (V1=1, V2=1)"

Commit message: First pass schematic done. Begin routing main board.
Parts:
- added C30: 33nF, pkl_dipol:C_0402, symbol device:C_Small
- added C32, C47, C48: 100nF, pkl_dipol:C_0402, symbol device:C_Small
- added C45: 10uF, pkl_dipol:C_0603, symbol device:C_Small
- added C49, C50: 10pF, pkl_dipol:C_0402, symbol device:C_Small
- added C51: 18pF, pkl_dipol:C_0402, symbol device:C_Small
- added J4: CTX TAG Connect, pkl_tag_connect:TC2030-NL_SMALL, symbol conn:Conn_02x03_Odd_Even
- added L21: 1k, pkl_dipol:L_0402, symbol device:Ferrite_Bead_Small
- added L22: 2.2nH, pkl_dipol:L_0402, symbol device:L_Small
- added OSC1: TYETBCSANF-32.000000, gkl_time:Oscilator_2.5x2.0, symbol gkl_time:TYETBCSANF-32.000000
- added R7: 10k, pkl_dipol:R_0402, symbol device:R
- added Y1: 32.768kHz, gkl_time:ABS05_32.768KHz Crystal, symbol device:Crystal_Small
Connections:
- net labels added: AUX_PWR_EN, BATTERY_VOLTAGE, CHARGE_STATUS, CLK, DIO, FLASH_CLK, FLASH_CS#, FLASH_DQ0, FLASH_DQ1, GPS_PPS, GPS_RX, GPS_TX, LED_A_BLUE, LED_A_GREEN, LED_A_RED, LED_B_BLUE, LED_B_GREEN, LED_B_RED, PP3V3_AUX, RESET, USER_BUTTON
- wire segments 251 -> 332
- no-connect marks 3 -> 5
Other:
- note added: "AIN11"
- note added: "EINT14"
- note added: "EINT15"
- note added: "EINT8"
- note added: "EINT9"
- note added: "SERCOM0.0\n"
- note added: "SERCOM1.0\n"
- note added: "SERCOM1.1"
- note added: "SERCOM1.2"
- note added: "SERCOM1.3"
- note added: "SERCOM5.0\n"
- note added: "SERCOM5.1\n"
- note added: "TC2.0"
- note added: "TC3.0"
- note added: "TC3.1"
- note added: "TC4.1\n"
- note added: "TCC1.0"
- note added: "TCC2.1"
- note added: "USB\n"

Commit message: Re-assigned IO pins. Added some extra filter as per Hardware guidelines.
Parts:
- added C57: 4.7pF, pkl_dipol:C_0402, symbol device:C_Small
- added L23, L24: 10nH, pkl_dipol:L_0402, symbol device:L_Small
- C22, C27: value 18pF -> 4.7pF
Connections:
- wire segments 332 -> 347
Other:
- note added: "EINT13\n"
- note added: "PAD\n\n 0\n\n 1\n\n 2\n\n 3"
- note added: "SERCOM PAD MAPPING"
- note added: "SERCOM5.2"
- note added: "SPI[0]\n\nMOSI\n\n~SS~\n\nMISO\n\nSCK"
- note added: "SPI[1]\n\nMISO\n\n~SS~\n\nMOSI\n\nSCK"
- note added: "TCC0.5"
- note added: "TCC1.1"
- note added: "TCC1.3\n"
- note added: "USART\n\nRX/TX\n\nRX\n\nRX/TX\n\nRX"
- note removed: "EINT9"
- note removed: "SERCOM0.0\n"
- note removed: "SERCOM5.1\n"
- note removed: "TC3.0"
- note removed: "TCC1.0"
- note removed: "TCC2.1"

Commit message: Added Vcore Cap. Missing from Microchips app note reference schematic
Parts:
- added C58: 1uF, pkl_dipol:C_0402, symbol device:C_Small
Connections:
- wire segments 347 -> 352
Changed lines of the file:
@@
 L device:C_Small C1
 U 1 1 5C407BF1
-P 4400 6200
-F 0 "C1" H 4250 6200 50  0000 C CNN
-F 1 "100nF" H 4250 6300 50  0000 C CNN
-F 2 "pkl_dipol:C_0402" H 4400 6200 50  0001 C CNN
-F 3 "~" H 4400 6200 50  0001 C CNN
-	1    4400 6200
+P 4600 6200
+F 0 "C1" H 4450 6200 50  0000 C CNN
+F 1 "100nF" H 4450 6300 50  0000 C CNN
+F 2 "pkl_dipol:C_0402" H 4600 6200 50  0001 C CNN
+F 3 "~" H 4600 6200 50  0001 C CNN
+	1    4600 6200
 	-1   0    0    1
 $EndComp
@@
 $EndComp
 Wire Wire Line
-	4050 6000 4400 6000
-Wire Wire Line
-	4400 6000 4400 5900
+	4050 6000 4600 6000
+Wire Wire Line
+	4600 6000 4600 5900
 $Comp
 L device:C_Small C2
@@
 $EndComp
 Wire Wire Line
-	4400 6300 4400 6350
+	4600 6300 4600 6350
 Wire Wire Line
 	5850 6350 5850 6400
@@
 L device:Ferrite_Bead_Small L18
 U 1 1 5C400786
-P 4950 5400
-F 0 "L18" H 4850 5354 50  0000 R CNN
-F 1 "1k" H 4850 5445 50  0000 R CNN
-F 2 "pkl_dipol:L_0402" V 4880 5400 50  0001 C CNN
-F 3 "~" H 4950 5400 50  0001 C CNN
-	1    4950 5400
+P 5100 5400
+F 0 "L18" H 5000 5354 50  0000 R CNN
+F 1 "1k" H 5000 5445 50  0000 R CNN
+F 2 "pkl_dipol:L_0402" V 5030 5400 50  0001 C CNN
+F 3 "~" H 5100 5400 50  0001 C CNN
+	1    5100 5400
 	1    0    0    -1
 $EndComp
@@
 	1    0    0    -1
 $EndComp
-Connection ~ 4400 6000
+Connection ~ 4600 6000
 Wire Wire Line
 	4050 5600 4150 5600
@@
 L power:GND #PWR0150
 U 1 1 5C473A30
-P 4750 6400
-F 0 "#PWR0150" H 4750 6150 50  0001 C CNN
-F 1 "GND" H 4755 6227 50  0000 C CNN
-F 2 "" H 4750 6400 50  0001 C CNN
-F 3 "" H 4750 6400 50  0001 C CNN
-	1    4750 6400
+P 4900 6400
+F 0 "#PWR0150" H 4900 6150 50  0001 C CNN
+F 1 "GND" H 4905 6227 50  0000 C CNN
+F 2 "" H 4900 6400 50  0001 C CNN
+F 3 "" H 4900 6400 50  0001 C CNN
+	1    4900 6400
 	1    0    0    -1
 $EndComp
@@
 L device:C_Small C45
 U 1 1 5C9F6851
-P 4750 6200
-F 0 "C45" H 4600 6200 50  0000 C CNN
-F 1 "10uF" H 4600 6300 50  0000 C CNN
-F 2 "pkl_dipol:C_0603" H 4750 6200 50  0001 C CNN
-F 3 "~" H 4750 6200 50  0001 C CNN
-	1    4750 6200
-	-1   0    0    1
-$EndComp
-Wire Wire Line
-	4750 6400 4750 6350
-Wire Wire Line
-	4750 6350 4400 6350
-Connection ~ 4750 6350
-Wire Wire Line
-	4750 6350 4750 6300
-Wire Wire Line
-	4750 6100 4750 6000
-Wire Wire Line
-	4750 5900 4400 5900
-Connection ~ 4400 5900
-Wire Wire Line
-	4400 6000 4400 6100
+P 4900 6200
+F 0 "C45" H 4750 6200 50  0000 C CNN
+F 1 "10uF" H 4750 6300 50  0000 C CNN
+F 2 "pkl_dipol:C_0603" H 4900 6200 50  0001 C CNN
+F 3 "~" H 4900 6200 50  0001 C CNN
+	1    4900 6200
+	-1   0    0    1
+$EndComp
+Wire Wire Line
+	4900 6400 4900 6350
+Wire Wire Line
+	4900 6350 4600 6350
+Connection ~ 4900 6350
+Wire Wire Line
+	4900 6350 4900 6300
+Wire Wire Line
+	4900 6100 4900 5900
+Wire Wire Line
+	4900 5900 4600 5900
+Wire Wire Line
+	4600 6000 4600 6100
 $Comp
 L device:C_Small C30
@@
 Wire Wire Line
 	4050 3900 4400 3900
-Connection ~ 4400 3900
 Wire Wire Line
 	4400 3900 4400 3700
@@
 CLK
 $Comp
-L power:AVDD #PWR0155
-U 1 1 5C59AD8E
-P 4750 5800
-F 0 "#PWR0155" H 4750 5650 50  0001 C CNN
-F 1 "AVDD" H 4753 5951 50  0000 C CNN
-F 2 "" H 4750 5800 50  0001 C CNN
-F 3 "" H 4750 5800 50  0001 C CNN
-	1    4750 5800
-	1    0    0    -1
-$EndComp
-Wire Wire Line
-	4750 5800 4750 5900
-$Comp
 L power:+3V3 #PWR0156
 U 1 1 5C5BC1F3
-P 4950 5150
-F 0 "#PWR0156" H 4950 5000 50  0001 C CNN
-F 1 "+3V3" H 4953 5301 50  0000 C CNN
-F 2 "" H 4950 5150 50  0001 C CNN
-F 3 "" H 4950 5150 50  0001 C CNN
-	1    4950 5150
+P 5100 5150
+F 0 "#PWR0156" H 5100 5000 50  0001 C CNN
+F 1 "+3V3" H 5103 5301 50  0000 C CNN
+F 2 "" H 5100 5150 50  0001 C CNN
+F 3 "" H 5100 5150 50  0001 C CNN
+	1    5100 5150
 	1    0    0    -1
 $EndComp
@@
 Wire Wire Line
 	6550 1800 8950 1800
-Connection ~ 4750 5900
-Wire Wire Line
-	4950 5150 4950 5300
-Wire Wire Line
-	4950 5500 4950 6000
-Wire Wire Line
-	4950 6000 4750 6000
-Connection ~ 4750 6000
-Wire Wire Line
-	4750 6000 4750 5900
-Wire Wire Line
-	4400 3900 4400 5900
+Wire Wire Line
+	5100 5150 5100 5300
+Wire Wire Line
+	5100 5500 5100 5900
+Wire Wire Line
+	5100 5900 4900 5900
+Connection ~ 4900 5900
 $Comp
 L device:C_Small C57
@@
 Wire Wire Line
 	1650 6650 1650 6000
-Text Notes 4000 7700 0    60   ~ 0
+Text Notes 3450 7700 0    60   ~ 0
 PAD\n\n 0\n\n 1\n\n 2\n\n 3
-Text Notes 4400 7700 0    60   ~ 0
+Text Notes 3850 7700 0    60   ~ 0
 USART\n\nRX/TX\n\nRX\n\nRX/TX\n\nRX
-Text Notes 5000 7700 0    60   ~ 0
+Text Notes 4450 7700 0    60   ~ 0
 SPI[0]\n\nMOSI\n\n~SS~\n\nMISO\n\nSCK
-Text Notes 5500 7700 0    60   ~ 0
+Text Notes 4950 7700 0    60   ~ 0
 SPI[1]\n\nMISO\n\n~SS~\n\nMOSI\n\nSCK
 Wire Notes Line
-	5850 6800 3900 6800
+	5300 6800 3350 6800
 Wire Notes Line
-	3900 7750 5850 7750
+	3350 7750 5300 7750
 Wire Notes Line
-	5850 6800 5850 7750
+	5300 6800 5300 7750
 Wire Notes Line
-	3900 6800 3900 7750
-Text Notes 4350 6750 0    60   ~ 0
+	3350 6800 3350 7750
+Text Notes 3800 6750 0    60   ~ 0
 SERCOM PAD MAPPING
+Wire Wire Line
+	4600 5900 4600 5600
+Wire Wire Line
+	4600 5600 4400 5600
+Wire Wire Line
+	4400 5600 4400 3900
+Connection ~ 4600 5900
+Connection ~ 4400 3900
+$Comp
+L power:AVDD #PWR0155
+U 1 1 5C351BF7
+P 4600 5500
+F 0 "#PWR0155" H 4600 5350 50  0001 C CNN
+F 1 "AVDD" H 4603 5651 50  0000 C CNN
+F 2 "" H 4600 5500 50  0001 C CNN
+F 3 "" H 4600 5500 50  0001 C CNN
+	1    4600 5500
+	1    0    0    -1
+$EndComp
+Wire Wire Line
+	4600 5600 4600 5500
+Connection ~ 4600 5600
+Wire Wire Line
+	4050 5900 4300 5900
+Wire Wire Line
+	4300 5900 4300 6100
+$Comp
+L device:C_Small C58
+U 1 1 5C3C154D
+P 4300 6200
+F 0 "C58" H 4150 6200 50  0000 C CNN
+F 1 "1uF" H 4150 6300 50  0000 C CNN
+F 2 "pkl_dipol:C_0402" H 4300 6200 50  0001 C CNN
+F 3 "~" H 4300 6200 50  0001 C CNN
+	1    4300 6200
+	-1   0    0    1
+$EndComp
+Wire Wire Line
+	4600 6350 4300 6350
+Wire Wire Line
+	4300 6350 4300 6300
+Connection ~ 4600 6350
 $EndSCHEMATC

Commit message: Checked RF filters with reference schematics. Updated all Part Numbers for BOM.
Parts:
- removed L5: 33nH, pkl_dipol:L_0402, symbol device:L_Small
- added C59: 4.7pF, pkl_dipol:C_0402, symbol device:C_Small
- A1: Mfg (none) -> Johanson Technology Inc.; PN (none) -> 0900AT43A0070E
- A2: Mfg (none) -> Johanson Technology Inc.; PN (none) -> 0433AT62A0020E
- C1, C2, C3, C32, C47, C48, C6: Mfg (none) -> Yageo; PN (none) -> CC0402KRX5R6BB104
- C10, C13, C34: Mfg (none) -> Murata Electronics North America; PN (none) -> GJM1555C1H220FB01D
- C12, C38: Mfg (none) -> Murata Electronics North America; PN (none) -> GJM1555C1H180FB01D
- C18, C36, C40, C7, C8: Mfg (none) -> Murata Electronics North America; PN (none) -> GJM1555C1H3R9CB01D
- C19: value 22pF -> 0R; Mfg (none) -> Vishay; PN (none) -> CRCW04020000Z0ED
- C20: Mfg (none) -> Murata Electronics North America; PN (none) -> GJM1555C1H8R2CB01D
- C22, C27, C57: Mfg (none) -> Murata Electronics North America; PN (none) -> GRM1555C1H4R7CA01D
- C23: Mfg (none) -> Yageo; PN (none) -> CC0402KRX7R9BB472
- C24: value 8.2pF -> 6.8pF; Mfg (none) -> Murata Electronics North America; PN (none) -> GRM1555C1H6R8CA01D
- C25: value DNP -> 2.7pF; Mfg (none) -> Murata Electronics North America; PN (none) -> GRM1555C1H2R7CZ01D
- C26: value 5.6pF -> 6.8pF; Mfg (none) -> Murata Electronics North America; PN (none) -> GRM1555C1H6R8CA01D
- C29: value 3.3pF -> DNP
- C30: Mfg (none) -> Yageo; PN (none) -> CC0402KRX7R7BB333
- C31, C42: Mfg (none) -> Yageo; PN (none) -> CC0402KRX7R8BB102
- C33: value 18pF -> 56pF; Mfg (none) -> Murata Electronics North America; PN (none) -> GRM1555C1H560JA01D
- C37: Mfg (none) -> Murata Electronics North America; PN (none) -> GJM1555C1H5R6BB01D
- C4: value 3.9pF -> 4.7pF; Mfg (none) -> Murata Electronics North America; PN (none) -> GRM1555C1H4R7CA01D
- C41: Mfg (none) -> Murata Electronics North America; PN (none) -> GJM1555C1H3R3CB01D
- C45: Mfg (none) -> Samsung Electro-Mechanics; PN (none) -> CL10A106MQ8NNNC
- C49, C50: Mfg (none) -> Murata Electronics North America; PN (none) -> GJM1555C1H100FB01D
- C5: value 3.9pF -> DNP
- C51: value 18pF -> 2.2pF; Mfg (none) -> Murata Electronics North America; PN (none) -> GRM1555C1H2R2CZ01D
- C58: Mfg (none) -> Yageo; PN (none) -> CC0402KRX5R6BB105
- L1, L10: value 2.2nH -> 18nH; Mfg (none) -> Murata Electronics North America; PN (none) -> LQG15HS18NJ02D
- L11, L12: Mfg (none) -> Murata Electronics North America; PN (none) -> LQW15AN11NJ00D
- L13, L14, L15, L16, L23, L24: Mfg (none) -> Murata Electronics North America; PN (none) -> LQW15AN10NJ00D
- L18, L21: Mfg (none) -> Murata Electronics North America; PN (none) -> BLM15AX102SN1D
- L2: Mfg (none) -> Murata Electronics North America; PN (none) -> LQW15AN2N2C10D
- L22: value 2.2nH -> 0R; Mfg (none) -> Vishay; PN (none) -> CRCW04020000Z0ED
- L3, L4: Mfg (none) -> Murata Electronics North America; PN (none) -> LQW15AN33NJ00D
- L6: value 33nH -> 82nH; Mfg (none) -> Murata Electronics North America; PN (none) -> LQG15HS82NJ02D
- L7: value 11nH -> 15nH; Mfg (none) -> Murata Electronics North America; PN (none) -> LQG15HS15NJ02D
- L8: value 10nH -> 12nH; Mfg (none) -> Murata Electronics North America; PN (none) -> LQG15HS12NJ02D
- L9: value 10nH -> 0R; Mfg (none) -> Vishay; PN (none) -> CRCW04020000Z0ED
- R7: Mfg (none) -> Yageo; PN (none) -> RC0402FR-0710KL
- U1, U4: Mfg (none) -> Skyworks Solutions Inc.; PN (none) -> SKY13373-460LF
- U8: Mfg (none) -> Microchip Technology; PN (none) -> ATSAMR34J18B-I/7JX
