File: hardware/v0.1a/USB.sch (KiCad schematic (older format))
At the start: 12 parts, among them J2 JST GH, U2 MCP73832, U3 NCP167

Commit message: First pass schematic done. Begin routing main board.
Parts:
- added C52: 100nF, pkl_dipol:C_0402, symbol device:C
- added C53: 1uF, pkl_dipol:C_0402, symbol device:C
- added Q1: FG6943010R, pkl_housings_sot:SOT-666, symbol gkl_mosfet:FG6943010R
- added R5: 10k, pkl_dipol:R_0402, symbol device:R
- added R6: 47k, pkl_dipol:R_Array_Concave_4x0603, symbol pkl_device:pkl_R4_Small
- added U6: NCP167, gkl_housings_son:X2SON_4_1.0x1.0mm, symbol gkl_pmic:NCP167
- C14, C16, C17: footprint pkl_dipol:C_0603 -> pkl_dipol:C_0402
- R1: value R -> 1k
- U2: footprint (none) -> pkl_housings_sot:SOT-23-5
- gave numbers to parts that had none: 1
Connections:
- net labels added: BATT_SENSE, PP3V3_AUX, PP3V3_AUX_EN
- wire segments 61 -> 106
Other:
- note added: "[0.2/0.25mm track/space]"

Commit message: Re-assigned IO pins. Added some extra filter as per Hardware guidelines.
Connections:
- net labels added: VBAT
Changed lines of the file:
@@
 $Comp
 L pkl_device:pkl_R4_Small R6
-U 2 1 5CE768A3
+U 4 1 5CE768A3
 P 8550 2650
 F 0 "R6" H 8609 2696 50  0000 L CNN
@@
 F 2 "pkl_dipol:R_Array_Concave_4x0603" H 8550 2650 60  0001 C CNN
 F 3 "" H 8550 2650 60  0000 C CNN
-	2    8550 2650
+	4    8550 2650
 	1    0    0    -1
 $EndComp
 $Comp
 L pkl_device:pkl_R4_Small R6
-U 1 1 5CE76947
+U 3 1 5CE76947
 P 8150 3450
 F 0 "R6" H 8209 3496 50  0000 L CNN
@@
 F 2 "pkl_dipol:R_Array_Concave_4x0603" H 8150 3450 60  0001 C CNN
 F 3 "" H 8150 3450 60  0000 C CNN
-	1    8150 3450
-	1    0    0    -1
+	3    8150 3450
+	1    0    0    1
 $EndComp
 $Comp
 L pkl_device:pkl_R4_Small R6
-U 3 1 5CE76991
+U 2 1 5CE76991
 P 9050 3200
 F 0 "R6" H 9109 3246 50  0000 L CNN
@@
 F 2 "pkl_dipol:R_Array_Concave_4x0603" H 9050 3200 60  0001 C CNN
 F 3 "" H 9050 3200 60  0000 C CNN
-	3    9050 3200
-	1    0    0    -1
+	2    9050 3200
+	1    0    0    1
 $EndComp
 $Comp
 L pkl_device:pkl_R4_Small R6
-U 4 1 5CE769DB
+U 1 1 5CE769DB
 P 9050 3500
 F 0 "R6" H 9109 3546 50  0000 L CNN
@@
 F 2 "pkl_dipol:R_Array_Concave_4x0603" H 9050 3500 60  0001 C CNN
 F 3 "" H 9050 3500 60  0000 C CNN
-	4    9050 3500
+	1    9050 3500
 	1    0    0    -1
 $EndComp
@@
 Wire Wire Line
 	7950 5250 5300 5250
+Text Label 5950 2000 0    60   ~ 0
+VBAT
 $EndSCHEMATC

Commit message: Small updates to the layout. Fixed up power planes. Passed DRC
Parts:
- added R8, R9: 5.1k, pkl_dipol:R_0402, symbol device:R
Connections:
- wire segments 106 -> 114
Changed lines of the file:
@@
 encoding utf-8
 Sheet 3 4
-Title ""
-Date ""
+Title "gpsLoggerLora"
+Date "2018-12-29"
 Rev ""
-Comp ""
+Comp "Gregory S Davill"
 Comment1 ""
 Comment2 ""
-Comment3 ""
-Comment4 ""
+Comment3 "Featuring a LoRa Tranciever"
+Comment4 "Simple GPS logger with low power features"
 $EndDescr
 Text Label 3850 3450 0    60   ~ 0
@@
 Text Label 5950 2000 0    60   ~ 0
 VBAT
+$Comp
+L device:R R8
+U 1 1 5C274F39
+P 2700 4250
+F 0 "R8" H 2770 4296 50  0000 L CNN
+F 1 "5.1k" H 2770 4205 50  0000 L CNN
+F 2 "pkl_dipol:R_0402" V 2630 4250 50  0001 C CNN
+F 3 "~" H 2700 4250 50  0001 C CNN
+	1    2700 4250
+	-1   0    0    -1
+$EndComp
+$Comp
+L device:R R9
+U 1 1 5C274F9F
+P 2850 4250
+F 0 "R9" H 2920 4296 50  0000 L CNN
+F 1 "5.1k" H 2920 4205 50  0000 L CNN
+F 2 "pkl_dipol:R_0402" V 2780 4250 50  0001 C CNN
+F 3 "~" H 2850 4250 50  0001 C CNN
+	1    2850 4250
+	1    0    0    -1
+$EndComp
+$Comp
+L power:GND #PWR?
+U 1 1 5C277E58
+P 2850 4700
+AR Path="/5C277E58" Ref="#PWR?"  Part="1"
+AR Path="/5C25E3B0/5C277E58" Ref="#PWR0161"  Part="1"
+F 0 "#PWR0161" H 2850 4450 50  0001 C CNN
+F 1 "GND" H 2853 4574 50  0000 C CNN
+F 2 "" H 2750 4350 50  0001 C CNN
+F 3 "" H 2850 4700 50  0001 C CNN
+	1    2850 4700
+	1    0    0    -1
+$EndComp
+Wire Wire Line
+	2700 4400 2700 4600
+Wire Wire Line
+	2700 4600 2850 4600
+Wire Wire Line
+	2850 4600 2850 4700
+Wire Wire Line
+	2850 4400 2850 4600
+Connection ~ 2850 4600
+Wire Wire Line
+	2050 3150 2700 3150
+Wire Wire Line
+	2700 3150 2700 4100
+Wire Wire Line
+	2050 3050 2850 3050
+Wire Wire Line
+	2850 3050 2850 4100
 $EndSCHEMATC

Commit message: Added TVS diode to USB input.
Parts:
- added U7: NUP2114, Package_TO_SOT_SMD:SOT-553, symbol gkl_misc:NUP2114
Connections:
- wire segments 114 -> 124
Changed lines of the file:
@@
 L device:C C?
 U 1 1 5C25E452
-P 2450 5650
+P 2450 4400
 AR Path="/5C25E452" Ref="C?"  Part="1"
 AR Path="/5C25E3B0/5C25E452" Ref="C9"  Part="1"
-F 0 "C9" H 2475 5750 50  0000 L CNN
-F 1 "10n" H 2475 5550 50  0000 L CNN
-F 2 "pkl_dipol:C_0402" H 2488 5500 30  0001 C CNN
-F 3 "" H 2450 5650 60  0000 C CNN
-	1    2450 5650
+F 0 "C9" H 2475 4500 50  0000 L CNN
+F 1 "10n" H 2475 4300 50  0000 L CNN
+F 2 "pkl_dipol:C_0402" H 2488 4250 30  0001 C CNN
+F 3 "" H 2450 4400 60  0000 C CNN
+	1    2450 4400
 	1    0    0    -1
 $EndComp
@@
 L power:GND #PWR?
 U 1 1 5C25E46E
-P 2450 5900
+P 2450 4750
 AR Path="/5C25E46E" Ref="#PWR?"  Part="1"
 AR Path="/5C25E3B0/5C25E46E" Ref="#PWR0119"  Part="1"
-F 0 "#PWR0119" H 2450 5650 50  0001 C CNN
-F 1 "GND" H 2453 5774 50  0000 C CNN
-F 2 "" H 2350 5550 50  0001 C CNN
-F 3 "" H 2450 5900 50  0001 C CNN
-	1    2450 5900
-	1    0    0    -1
-$EndComp
-Wire Wire Line
-	2450 5900 2450 5800
+F 0 "#PWR0119" H 2450 4500 50  0001 C CNN
+F 1 "GND" H 2453 4624 50  0000 C CNN
+F 2 "" H 2350 4400 50  0001 C CNN
+F 3 "" H 2450 4750 50  0001 C CNN
+	1    2450 4750
+	1    0    0    -1
+$EndComp
+Wire Wire Line
+	2450 4750 2450 4650
 $Comp
 L power:GND #PWR?
@@
 $EndComp
 Wire Notes Line
-	2950 3400 2950 3600
+	5150 5500 5150 5700
 Wire Notes Line
-	2950 3600 3050 3600
+	5150 5700 5250 5700
 Wire Notes Line
-	3050 3400 2950 3400
+	5250 5500 5150 5500
 Wire Notes Line
-	3050 3750 3200 3750
+	5250 5850 5400 5850
 Wire Notes Line
-	3050 3400 3050 3750
-Text Notes 3200 3750 0    60   ~ 0
+	5250 5500 5250 5850
+Text Notes 5400 5850 0    60   ~ 0
 Route as 90-Ohm diff pair
 Wire Notes Line
@@
 Wire Wire Line
 	2150 3350 2150 3450
-Connection ~ 2150 3450
 Wire Wire Line
 	2050 3650 2150 3650
@@
 Wire Wire Line
 	2150 3550 2050 3550
-Connection ~ 2150 3550
 Connection ~ 2450 2550
 Wire Wire Line
@@
 Connection ~ 2450 2850
 Wire Wire Line
-	2450 2850 2450 5500
+	2450 2850 2450 4100
 Wire Wire Line
 	1550 5450 1550 5550
@@
 	9100 5550 4900 5550
 Wire Wire Line
-	4900 5550 4900 3450
+	4900 5550 4900 4300
 Wire Wire Line
 	2150 3450 4900 3450
 Wire Wire Line
-	4800 3550 4800 5650
+	4800 3550 4800 4100
 Wire Wire Line
 	4800 5650 9100 5650
@@
 Wire Wire Line
 	5550 4350 6100 4350
-Text Notes 3200 3850 0    60   ~ 0
+Text Notes 5400 5950 0    60   ~ 0
 [0.2/0.25mm track/space]
 Wire Wire Line
@@
 L device:R R8
 U 1 1 5C274F39
-P 2700 4250
-F 0 "R8" H 2770 4296 50  0000 L CNN
-F 1 "5.1k" H 2770 4205 50  0000 L CNN
-F 2 "pkl_dipol:R_0402" V 2630 4250 50  0001 C CNN
-F 3 "~" H 2700 4250 50  0001 C CNN
-	1    2700 4250
+P 2950 5600
+F 0 "R8" H 3020 5646 50  0000 L CNN
+F 1 "5.1k" H 3020 5555 50  0000 L CNN
+F 2 "pkl_dipol:R_0402" V 2880 5600 50  0001 C CNN
+F 3 "~" H 2950 5600 50  0001 C CNN
+	1    2950 5600
 	-1   0    0    -1
 $EndComp
@@
 L device:R R9
 U 1 1 5C274F9F
-P 2850 4250
-F 0 "R9" H 2920 4296 50  0000 L CNN
-F 1 "5.1k" H 2920 4205 50  0000 L CNN
-F 2 "pkl_dipol:R_0402" V 2780 4250 50  0001 C CNN
-F 3 "~" H 2850 4250 50  0001 C CNN
-	1    2850 4250
+P 3100 5600
+F 0 "R9" H 3170 5646 50  0000 L CNN
+F 1 "5.1k" H 3170 5555 50  0000 L CNN
+F 2 "pkl_dipol:R_0402" V 3030 5600 50  0001 C CNN
+F 3 "~" H 3100 5600 50  0001 C CNN
+	1    3100 5600
 	1    0    0    -1
 $EndComp
@@
 L power:GND #PWR?
 U 1 1 5C277E58
-P 2850 4700
+P 3100 6050
 AR Path="/5C277E58" Ref="#PWR?"  Part="1"
 AR Path="/5C25E3B0/5C277E58" Ref="#PWR0161"  Part="1"
-F 0 "#PWR0161" H 2850 4450 50  0001 C CNN
-F 1 "GND" H 2853 4574 50  0000 C CNN
-F 2 "" H 2750 4350 50  0001 C CNN
-F 3 "" H 2850 4700 50  0001 C CNN
-	1    2850 4700
-	1    0    0    -1
-$EndComp
-Wire Wire Line
-	2700 4400 2700 4600
-Wire Wire Line
-	2700 4600 2850 4600
-Wire Wire Line
-	2850 4600 2850 4700
-Wire Wire Line
-	2850 4400 2850 4600
-Connection ~ 2850 4600
-Wire Wire Line
-	2050 3150 2700 3150
-Wire Wire Line
-	2700 3150 2700 4100
-Wire Wire Line
-	2050 3050 2850 3050
-Wire Wire Line
-	2850 3050 2850 4100
+F 0 "#PWR0161" H 3100 5800 50  0001 C CNN
+F 1 "GND" H 3103 5924 50  0000 C CNN
+F 2 "" H 3000 5700 50  0001 C CNN
+F 3 "" H 3100 6050 50  0001 C CNN
+	1    3100 6050
+	1    0    0    -1
+$EndComp
+Wire Wire Line
+	2950 5750 2950 5950
+Wire Wire Line
+	2950 5950 3100 5950
+Wire Wire Line
+	3100 5950 3100 6050
+Wire Wire Line
+	3100 5750 3100 5950
+Connection ~ 3100 5950
+Wire Wire Line
+	2050 3150 2950 3150
+Wire Wire Line
+	2950 3150 2950 5450
+Wire Wire Line
+	2050 3050 3100 3050
+Wire Wire Line
+	3100 3050 3100 5450
+Connection ~ 2150 3450
+Connection ~ 2150 3550
+$Comp
+L gkl_misc:NUP2114 U7
+U 1 1 5C287FF8
+P 3850 4050
+F 0 "U7" H 3875 4268 50  0000 C CNN
+F 1 "NUP2114" H 3875 4177 50  0000 C CNN
+F 2 "Package_TO_SOT_SMD:SOT-553" H 3850 4200 50  0001 C CNN
+F 3 "" H 3850 4200 50  0001 C CNN
+	1    3850 4050
+	1    0    0    -1
+$EndComp
+Wire Wire Line
+	3400 4100 2450 4100
+Connection ~ 2450 4100
+Wire Wire Line
+	2450 4100 2450 4250
+Wire Wire Line
+	2450 4650 2750 4650
+Wire Wire Line
+	2750 4650 2750 4300
+Wire Wire Line
+	2750 4300 3400 4300
+Connection ~ 2450 4650
+Wire Wire Line
+	2450 4650 2450 4550
+Wire Wire Line
+	4350 4100 4800 4100
+Connection ~ 4800 4100
+Wire Wire Line
+	4800 4100 4800 5650
+Wire Wire Line
+	4350 4300 4900 4300
+Connection ~ 4900 4300
+Wire Wire Line
+	4900 4300 4900 3450
 $EndSCHEMATC

Commit message: Checked RF filters with reference schematics. Updated all Part Numbers for BOM.
Parts:
- C11, C15, C52: Mfg (none) -> Yageo; PN (none) -> CC0402KRX5R6BB104
- C14, C16, C17, C53: Mfg (none) -> Yageo; PN (none) -> CC0402KRX5R6BB105
- C9: Mfg (none) -> Yageo; PN (none) -> CC0402KRX7R8BB103
- J1: Mfg (none) -> Amphenol ICC (FCI); PN (none) -> 10132328-10011LF
- J2: Mfg (none) -> JST Sales America Inc.; PN (none) -> BM02B-GHS-TBT(LF)(SN)(N)
- L17: Mfg (none) -> Murata Electronics North America; PN (none) -> BLM15AX102SN1D
- Q1: Mfg (none) -> Panasonic Electronic Components; PN (none) -> FG6943010R
- R1: value 1k -> 10k; Mfg (none) -> Yageo; PN (none) -> RC0603FR-0710KL
- R5: Mfg (none) -> Yageo; PN (none) -> RC0402FR-0710KL
- R6: Mfg (none) -> Panasonic Electronic Components; PN (none) -> EXB-38V473JV
- R8, R9: Mfg (none) -> Yageo; PN (none) -> RC0402FR-075K1L
- U3, U6: Mfg (none) -> ON Semiconductor; PN (none) -> NCP167AMX330TBG
- U7: Mfg (none) -> ON Semiconductor; PN (none) -> NUP2114UPXV5T1G
Changed lines of the file:
@@
 F 2 "pkl_dipol:C_0402" H 2488 4250 30  0001 C CNN
 F 3 "" H 2450 4400 60  0000 C CNN
+F 4 "Yageo" H 0   0   50  0001 C CNN "Mfg"
+F 5 "CC0402KRX7R8BB103" H 0   0   50  0001 C CNN "PN"
 	1    2450 4400
 	1    0    0    -1
@@
 F 2 "gkl_housings_son:X2SON_4_1.0x1.0mm" H 6500 3500 50  0001 C CNN
 F 3 "http://www.onsemi.com/pub/Collateral/NCP167-D.PDF" H 6550 3400 50  0001 C CNN
+F 4 "ON Semiconductor" H 0   0   50  0001 C CNN "Mfg"
+F 5 "NCP167AMX330TBG" H 0   0   50  0001 C CNN "PN"
 	1    6550 3150
 	1    0    0    -1
@@
 F 2 "pkl_dipol:C_0402" H 5538 2300 30  0001 C CNN
 F 3 "" H 5500 2450 60  0000 C CNN
+F 4 "Yageo" H 0   0   50  0001 C CNN "Mfg"
+F 5 "CC0402KRX5R6BB105" H 0   0   50  0001 C CNN "PN"
 	1    5500 2450
 	1    0    0    -1
@@
 F 2 "" H 9600 2000 50  0001 C CNN
 F 3 "~" H 9600 2000 50  0001 C CNN
+F 4 "JST Sales America Inc." H 0   0   50  0001 C CNN "Mfg"
+F 5 "BM02B-GHS-TBT(LF)(SN)(N)" H 0   0   50  0001 C CNN "PN"
 	1    9600 2000
 	-1   0    0    -1
@@
 P 4100 2600
 F 0 "R1" H 4170 2646 50  0000 L CNN
-F 1 "1k" H 4170 2555 50  0000 L CNN
+F 1 "10k" H 4170 2555 50  0000 L CNN
 F 2 "pkl_dipol:R_0603" V 4030 2600 50  0001 C CNN
 F 3 "~" H 4100 2600 50  0001 C CNN
+F 4 "Yageo" H 0   0   50  0001 C CNN "Mfg"
+F 5 "RC0603FR-0710KL" H 0   0   50  0001 C CNN "PN"
 	1    4100 2600
 	1    0    0    -1
@@
 F 2 "pkl_dipol:C_0402" H 6038 3400 30  0001 C CNN
 F 3 "" H 6000 3550 60  0000 C CNN
+F 4 "Yageo" H 0   0   50  0001 C CNN "Mfg"
+F 5 "CC0402KRX5R6BB104" H 0   0   50  0001 C CNN "PN"
 	1    6000 3550
 	1    0    0    -1
@@
 F 2 "pkl_dipol:C_0402" H 3788 2200 30  0001 C CNN
 F 3 "" H 3750 2350 60  0000 C CNN
+F 4 "Yageo" H 0   0   50  0001 C CNN "Mfg"
+F 5 "CC0402KRX5R6BB105" H 0   0   50  0001 C CNN "PN"
 	1    3750 2350
 	1    0    0    -1
@@
 F 2 "pkl_dipol:C_0402" H 3438 2200 30  0001 C CNN
 F 3 "" H 3400 2350 60  0000 C CNN
+F 4 "Yageo" H 0   0   50  0001 C CNN "Mfg"
+F 5 "CC0402KRX5R6BB104" H 0   0   50  0001 C CNN "PN"
 	1    3400 2350
 	1    0    0    -1
@@
 F 2 "pkl_dipol:L_0402" V 2930 2000 50  0001 C CNN
 F 3 "~" H 3000 2000 50  0001 C CNN
+F 4 "Murata Electronics North America" H 0   0   50  0001 C CNN "Mfg"
+F 5 "BLM15AX102SN1D" H 0   0   50  0001 C CNN "PN"
 	1    3000 2000
 	0    1    1    0
@@
 F 2 "pkl_dipol:C_0402" H 7388 3150 30  0001 C CNN
 F 3 "" H 7350 3300 60  0000 C CNN
+F 4 "Yageo" H 0   0   50  0001 C CNN "Mfg"
+F 5 "CC0402KRX5R6BB105" H 0   0   50  0001 C CNN "PN"
 	1    7350 3300
 	1    0    0    -1
@@
 F 2 "gkl_conn:usbc_vert_10132328" H 1600 3850 50  0001 C CNN
 F 3 "http://www.usb.org/developers/docs/usb_31_033017.zip" H 1600 3850 50  0001 C CNN
+F 4 "Amphenol ICC (FCI)" H 0   0   50  0001 C CNN "Mfg"
+F 5 "10132328-10011LF" H 0   0   50  0001 C CNN "PN"
 	1    1450 3850
 	1    0    0    -1
@@
 F 2 "gkl_housings_son:X2SON_4_1.0x1.0mm" H 6500 4600 50  0001 C CNN
 F 3 "http://www.onsemi.com/pub/Collateral/NCP167-D.PDF" H 6550 4500 50  0001 C CNN
+F 4 "ON Semiconductor" H 0   0   50  0001 C CNN "Mfg"
+F 5 "NCP167AMX330TBG" H 0   0   50  0001 C CNN "PN"
 	1    6550 4250
 	1    0    0    -1
@@
 F 2 "pkl_dipol:C_0402" H 6038 4600 30  0001 C CNN
 F 3 "" H 6000 4750 60  0000 C CNN
+F 4 "Yageo" H 0   0   50  0001 C CNN "Mfg"
+F 5 "CC0402KRX5R6BB104" H 0   0   50  0001 C CNN "PN"
 	1    6000 4750
 	1    0    0    -1
@@
 F 2 "pkl_dipol:C_0402" H 7388 4300 30  0001 C CNN
 F 3 "" H 7350 4450 60  0000 C CNN
+F 4 "Yageo" H 0   0   50  0001 C CNN "Mfg"
+F 5 "CC0402KRX5R6BB105" H 0   0   50  0001 C CNN "PN"
 	1    7350 4450
 	1    0    0    -1
@@
 F 2 "pkl_dipol:R_0402" V 5480 4700 50  0001 C CNN
 F 3 "~" H 5550 4700 50  0001 C CNN
+F 4 "Yageo" H 0   0   50  0001 C CNN "Mfg"
+F 5 "RC0402FR-0710KL" H 0   0   50  0001 C CNN "PN"
 	1    5550 4700
 	1    0    0    -1
@@
 F 2 "pkl_housings_sot:SOT-666" H 8650 3300 29  0001 C CNN
 F 3 "" H 8450 3200 60  0000 C CNN
+F 4 "Panasonic Electronic Components" H 0   0   50  0001 C CNN "Mfg"
+F 5 "FG6943010R" H 0   0   50  0001 C CNN "PN"
 	1    8450 3200
 	1    0    0    -1
@@
 F 2 "pkl_housings_sot:SOT-666" H 9141 2809 29  0001 L CNN
 F 3 "" H 8950 2900 60  0000 C CNN
+F 4 "Panasonic Electronic Components" H 0   0   50  0001 C CNN "Mfg"
+F 5 "FG6943010R" H 0   0   50  0001 C CNN "PN"
 	2    8950 2900
 	1    0    0    -1
@@
 F 2 "pkl_dipol:R_Array_Concave_4x0603" H 8550 2650 60  0001 C CNN
 F 3 "" H 8550 2650 60  0000 C CNN
+F 4 "Panasonic Electronic Components" H 0   0   50  0001 C CNN "Mfg"
+F 5 "EXB-38V473JV" H 0   0   50  0001 C CNN "PN"
 	4    8550 2650
 	1    0    0    -1
@@
 F 2 "pkl_dipol:R_Array_Concave_4x0603" H 8150 3450 60  0001 C CNN
 F 3 "" H 8150 3450 60  0000 C CNN
+F 4 "Panasonic Electronic Components" H 0   0   50  0001 C CNN "Mfg"
+F 5 "EXB-38V473JV" H 0   0   50  0001 C CNN "PN"
 	3    8150 3450
 	1    0    0    1
@@
 F 2 "pkl_dipol:R_Array_Concave_4x0603" H 9050 3200 60  0001 C CNN
 F 3 "" H 9050 3200 60  0000 C CNN
+F 4 "Panasonic Electronic Components" H 0   0   50  0001 C CNN "Mfg"
+F 5 "EXB-38V473JV" H 0   0   50  0001 C CNN "PN"
 	2    9050 3200
 	1    0    0    1
@@
 F 2 "pkl_dipol:R_Array_Concave_4x0603" H 9050 3500 60  0001 C CNN
 F 3 "" H 9050 3500 60  0000 C CNN
+F 4 "Panasonic Electronic Components" H 0   0   50  0001 C CNN "Mfg"
+F 5 "EXB-38V473JV" H 0   0   50  0001 C CNN "PN"
 	1    9050 3500
 	1    0    0    -1
@@
 F 2 "pkl_dipol:R_0402" V 2880 5600 50  0001 C CNN
 F 3 "~" H 2950 5600 50  0001 C CNN
+F 4 "Yageo" H 0   0   50  0001 C CNN "Mfg"
+F 5 "RC0402FR-075K1L" H 0   0   50  0001 C CNN "PN"
 	1    2950 5600
 	-1   0    0    -1
@@
 F 2 "pkl_dipol:R_0402" V 3030 5600 50  0001 C CNN
 F 3 "~" H 3100 5600 50  0001 C CNN
+F 4 "Yageo" H 0   0   50  0001 C CNN "Mfg"
+F 5 "RC0402FR-075K1L" H 0   0   50  0001 C CNN "PN"
 	1    3100 5600
 	1    0    0    -1
@@
 F 2 "Package_TO_SOT_SMD:SOT-553" H 3850 4200 50  0001 C CNN
 F 3 "" H 3850 4200 50  0001 C CNN
+F 4 "ON Semiconductor" H 0   0   50  0001 C CNN "Mfg"
+F 5 "NUP2114UPXV5T1G" H 0   0   50  0001 C CNN "PN"
 	1    3850 4050
 	1    0    0    -1
