File: hardware/v0.1a/memio.sch (KiCad schematic (older format))
At the start: 1 part, among them U5 MT25QL256ABA8E12

Commit message: First pass schematic done. Begin routing main board.
Parts:
- added C43, C44, C54, C55, C56: 100nF, pkl_dipol:C_0402, symbol device:C_Small
- added C46: 10uF, pkl_dipol:C_0603, symbol device:C_Small
- added D1, D2: LED_ARGB, symbol device:LED_ARGB
- added J3: DF12 - 10P, gkl_conn:DF12(3.0)-10DP-0.5V(86), symbol conn:Conn_02x05_Odd_Even
- added L19, L20: 1k, pkl_dipol:L_0402, symbol device:Ferrite_Bead_Small
- added R2, R3, R4: 100R, pkl_dipol:R_Array_Concave_4x0603, symbol pkl_device:pkl_R4_Small
- added SW1: SW_Push, symbol Switch:SW_Push
Connections:
- net labels added: DQ0, DQ1, FLASH_CLK, FLASH_CS#, GPS_PPS, GPS_RXD, GPS_TXD, LED_A_BLUE, LED_A_GREEN, LED_A_RED, LED_B_BLUE, LED_B_GREEN, LED_B_RED, PP3V3_AUX, USER_BUTTON
- net labels removed: +3V3
- wire segments 4 -> 86
Other:
- note added: "Status A\n"
- note added: "Status B\n"

Commit message: Re-assigned IO pins. Added some extra filter as per Hardware guidelines.
Parts:
- D1, D2: footprint (none) -> gkl_led:0404LED_RGB
Changed lines of the file:
@@
 F 0 "D1" H 4300 5497 50  0000 C CNN
 F 1 "LED_ARGB" H 4300 5406 50  0000 C CNN
-F 2 "" H 4300 4950 50  0001 C CNN
+F 2 "gkl_led:0404LED_RGB" H 4300 4950 50  0001 C CNN
 F 3 "~" H 4300 4950 50  0001 C CNN
 	1    4300 5000
@@
 F 0 "D2" H 4300 6397 50  0000 C CNN
 F 1 "LED_ARGB" H 4300 6306 50  0000 C CNN
-F 2 "" H 4300 5850 50  0001 C CNN
+F 2 "gkl_led:0404LED_RGB" H 4300 5850 50  0001 C CNN
 F 3 "~" H 4300 5850 50  0001 C CNN
 	1    4300 5900

Commit message: Small updates to the layout. Fixed up power planes. Passed DRC
Parts:
- C43: value 100nF -> 1uF
Connections:
- net labels added: +3V3
- wire segments 86 -> 88
Other:
- note added: "Pin 10: \nVbat supply of GPS"
- note added: "RGB Values may \nnot align with this symbol"
Changed lines of the file:
@@
 encoding utf-8
 Sheet 4 4
-Title ""
-Date ""
+Title "gpsLoggerLora"
+Date "2018-12-29"
 Rev ""
-Comp ""
+Comp "Gregory S Davill"
 Comment1 ""
 Comment2 ""
-Comment3 ""
-Comment4 ""
+Comment3 "Featuring a LoRa Tranciever"
+Comment4 "Simple GPS logger with low power features"
 $EndDescr
 $Comp
@@
 P 3700 5200
 F 0 "R3" V 3600 5050 50  0000 C CNN
-F 1 "100R" V 3600 5300 50  0000 C CNN
+F 1 "100R" V 3600 5350 50  0000 C CNN
 F 2 "pkl_dipol:R_Array_Concave_4x0603" H 3700 5200 60  0001 C CNN
 F 3 "" H 3700 5200 60  0000 C CNN
@@
 P 3700 5700
 F 0 "R3" V 3600 5550 50  0000 C CNN
-F 1 "100R" V 3600 5800 50  0000 C CNN
+F 1 "100R" V 3600 5850 50  0000 C CNN
 F 2 "pkl_dipol:R_Array_Concave_4x0603" H 3700 5700 60  0001 C CNN
 F 3 "" H 3700 5700 60  0000 C CNN
@@
 U 2 1 5C26DE81
 P 3700 6100
-F 0 "R2" V 3800 5950 50  0000 C CNN
-F 1 "100R" V 3750 6250 50  0000 C CNN
+F 0 "R2" V 3600 5950 50  0000 C CNN
+F 1 "100R" V 3600 6250 50  0000 C CNN
 F 2 "pkl_dipol:R_Array_Concave_4x0603" H 3700 6100 60  0001 C CNN
 F 3 "" H 3700 6100 60  0000 C CNN
@@
 L pkl_device:pkl_R4_Small R2
 U 3 1 5C26EB4D
-P 3700 7150
-F 0 "R2" V 3800 7000 50  0000 C CNN
-F 1 "100R" V 3750 7300 50  0000 C CNN
-F 2 "pkl_dipol:R_Array_Concave_4x0603" H 3700 7150 60  0001 C CNN
-F 3 "" H 3700 7150 60  0000 C CNN
-	3    3700 7150
+P 3700 6950
+F 0 "R2" V 3800 6800 50  0000 C CNN
+F 1 "100R" V 3750 7100 50  0000 C CNN
+F 2 "pkl_dipol:R_Array_Concave_4x0603" H 3700 6950 60  0001 C CNN
+F 3 "" H 3700 6950 60  0000 C CNN
+	3    3700 6950
 	0    1    1    0
 $EndComp
@@
 P 4500 1850
 F 0 "C43" H 4592 1896 50  0000 L CNN
-F 1 "100nF" H 4592 1805 50  0000 L CNN
+F 1 "1uF" H 4592 1805 50  0000 L CNN
 F 2 "pkl_dipol:C_0402" H 4500 1850 50  0001 C CNN
 F 3 "~" H 4500 1850 50  0001 C CNN
@@
 L Switch:SW_Push SW1
 U 1 1 5CEEE3F1
-P 4300 7150
-F 0 "SW1" H 4300 7435 50  0000 C CNN
-F 1 "SW_Push" H 4300 7344 50  0000 C CNN
-F 2 "" H 4300 7350 50  0001 C CNN
-F 3 "" H 4300 7350 50  0001 C CNN
-	1    4300 7150
-	1    0    0    -1
-$EndComp
-Wire Wire Line
-	4500 7150 4700 7150
-Wire Wire Line
-	4700 7150 4700 7550
-Wire Wire Line
-	4100 7150 3800 7150
+P 4300 6950
+F 0 "SW1" H 4300 7235 50  0000 C CNN
+F 1 "SW_Push" H 4300 7144 50  0000 C CNN
+F 2 "" H 4300 7150 50  0001 C CNN
+F 3 "" H 4300 7150 50  0001 C CNN
+	1    4300 6950
+	1    0    0    -1
+$EndComp
+Wire Wire Line
+	4500 6950 4700 6950
+Wire Wire Line
+	4700 6950 4700 7350
+Wire Wire Line
+	4100 6950 3800 6950
 $Comp
 L device:C_Small C56
 U 1 1 5CEF2AA6
-P 3350 7400
-F 0 "C56" H 3442 7446 50  0000 L CNN
-F 1 "100nF" H 3442 7355 50  0000 L CNN
-F 2 "pkl_dipol:C_0402" H 3350 7400 50  0001 C CNN
-F 3 "~" H 3350 7400 50  0001 C CNN
-	1    3350 7400
+P 3350 7200
+F 0 "C56" H 3442 7246 50  0000 L CNN
+F 1 "100nF" H 3442 7155 50  0000 L CNN
+F 2 "pkl_dipol:C_0402" H 3350 7200 50  0001 C CNN
+F 3 "~" H 3350 7200 50  0001 C CNN
+	1    3350 7200
 	1    0    0    -1
 $EndComp
@@
 L power:GND #PWR0151
 U 1 1 5CEF2AAC
-P 3350 7550
-F 0 "#PWR0151" H 3350 7300 50  0001 C CNN
-F 1 "GND" H 3353 7424 50  0000 C CNN
-F 2 "" H 3250 7200 50  0001 C CNN
-F 3 "" H 3350 7550 50  0001 C CNN
-	1    3350 7550
-	-1   0    0    -1
-$EndComp
-Wire Wire Line
-	3350 7550 3350 7500
-Wire Wire Line
-	3350 7300 3350 7150
-Wire Wire Line
-	3600 7150 3350 7150
-Wire Wire Line
-	3350 7150 2500 7150
-Connection ~ 3350 7150
+P 3350 7350
+F 0 "#PWR0151" H 3350 7100 50  0001 C CNN
+F 1 "GND" H 3353 7224 50  0000 C CNN
+F 2 "" H 3250 7000 50  0001 C CNN
+F 3 "" H 3350 7350 50  0001 C CNN
+	1    3350 7350
+	-1   0    0    -1
+$EndComp
+Wire Wire Line
+	3350 7350 3350 7300
+Wire Wire Line
+	3350 7100 3350 6950
+Wire Wire Line
+	3600 6950 3350 6950
+Wire Wire Line
+	3350 6950 2500 6950
+Connection ~ 3350 6950
 $Comp
 L power:GND #PWR0152
 U 1 1 5CEFB4F0
-P 4700 7550
-F 0 "#PWR0152" H 4700 7300 50  0001 C CNN
-F 1 "GND" H 4703 7424 50  0000 C CNN
-F 2 "" H 4600 7200 50  0001 C CNN
-F 3 "" H 4700 7550 50  0001 C CNN
-	1    4700 7550
-	-1   0    0    -1
-$EndComp
-Text HLabel 2500 7150 0    60   Input ~ 0
+P 4700 7350
+F 0 "#PWR0152" H 4700 7100 50  0001 C CNN
+F 1 "GND" H 4703 7224 50  0000 C CNN
+F 2 "" H 4600 7000 50  0001 C CNN
+F 3 "" H 4700 7350 50  0001 C CNN
+	1    4700 7350
+	-1   0    0    -1
+$EndComp
+Text HLabel 2500 6950 0    60   Input ~ 0
 USER_BUTTON
 Wire Wire Line
@@
 Wire Wire Line
 	2500 3300 3700 3300
+Wire Wire Line
+	8000 4000 6400 4000
+Wire Wire Line
+	6400 4000 6400 3050
+$Comp
+L power:+3V3 #PWR0162
+U 1 1 5C279185
+P 6400 3050
+F 0 "#PWR0162" H 6400 2900 50  0001 C CNN
+F 1 "+3V3" H 6403 3201 50  0000 C CNN
+F 2 "" H 6400 3050 50  0001 C CNN
+F 3 "" H 6400 3050 50  0001 C CNN
+	1    6400 3050
+	1    0    0    -1
+$EndComp
+Text Notes 6950 4250 0    60   ~ 0
+Pin 10: \nVbat supply of GPS
+Text Notes 4600 5450 0    60   ~ 0
+RGB Values may \nnot align with this symbol
 $EndSCHEMATC

Commit message: Checked RF filters with reference schematics. Updated all Part Numbers for BOM.
Parts:
- C43: Mfg (none) -> Yageo; PN (none) -> CC0402KRX5R6BB105
- C44, C54, C55, C56: Mfg (none) -> Yageo; PN (none) -> CC0402KRX5R6BB104
- C46: Mfg (none) -> Samsung Electro-Mechanics; PN (none) -> CL10A106MQ8NNNC
- D1, D2: Mfg (none) -> OSRAM Opto Semiconductors Inc.; PN (none) -> LRTBR48G-P9Q7-1+R7S5-26+N5P-68-R33-ZB
- J3: Mfg (none) -> Hirose Electric Co Ltd; PN (none) -> DF12(3.0)-10DP-0.5V(86)
- L19, L20: Mfg (none) -> Murata Electronics North America; PN (none) -> BLM15AX102SN1D
- R2, R3, R4: Mfg (none) -> Panasonic Electronic Components; PN (none) -> EXB-38V101JV
- SW1: Mfg (none) -> Panasonic Electronic Components; PN (none) -> EVQ-P1D05M
- U5: Mfg (none) -> Micron Technology Inc.; PN (none) -> MT25QL256ABA8E12-1SIT TR
Changed lines of the file:
@@
 F 2 "gkl_housings_bga:T-PBGA-24_6.0x8.0mm_Layout5x5_P1.0mm" H 4300 3750 50  0001 C CNN
 F 3 "" H 4300 3750 50  0001 C CNN
+F 4 "Micron Technology Inc." H 0   0   50  0001 C CNN "Mfg"
+F 5 "MT25QL256ABA8E12-1SIT TR" H 0   0   50  0001 C CNN "PN"
 	1    4300 3250
 	1    0    0    -1
@@
 F 2 "gkl_led:0404LED_RGB" H 4300 4950 50  0001 C CNN
 F 3 "~" H 4300 4950 50  0001 C CNN
+F 4 "OSRAM Opto Semiconductors Inc." H 0   0   50  0001 C CNN "Mfg"
+F 5 "LRTBR48G-P9Q7-1+R7S5-26+N5P-68-R33-ZB" H 0   0   50  0001 C CNN "PN"
 	1    4300 5000
 	1    0    0    -1
@@
 F 2 "gkl_led:0404LED_RGB" H 4300 5850 50  0001 C CNN
 F 3 "~" H 4300 5850 50  0001 C CNN
+F 4 "OSRAM Opto Semiconductors Inc." H 0   0   50  0001 C CNN "Mfg"
+F 5 "LRTBR48G-P9Q7-1+R7S5-26+N5P-68-R33-ZB" H 0   0   50  0001 C CNN "PN"
 	1    4300 5900
 	1    0    0    -1
@@
 F 2 "pkl_dipol:R_Array_Concave_4x0603" H 3700 4800 60  0001 C CNN
 F 3 "" H 3700 4800 60  0000 C CNN
+F 4 "Panasonic Electronic Components" H 0   0   50  0001 C CNN "Mfg"
+F 5 "EXB-38V101JV" H 0   0   50  0001 C CNN "PN"
 	1    3700 4800
 	0    1    1    0
@@
 F 2 "pkl_dipol:R_Array_Concave_4x0603" H 3700 5000 60  0001 C CNN
 F 3 "" H 3700 5000 60  0000 C CNN
+F 4 "Panasonic Electronic Components" H 0   0   50  0001 C CNN "Mfg"
+F 5 "EXB-38V101JV" H 0   0   50  0001 C CNN "PN"
 	2    3700 5000
 	0    1    1    0
@@
 F 2 "pkl_dipol:R_Array_Concave_4x0603" H 3700 5200 60  0001 C CNN
 F 3 "" H 3700 5200 60  0000 C CNN
+F 4 "Panasonic Electronic Components" H 0   0   50  0001 C CNN "Mfg"
+F 5 "EXB-38V101JV" H 0   0   50  0001 C CNN "PN"
 	3    3700 5200
 	0    1    1    0
@@
 F 2 "pkl_dipol:R_Array_Concave_4x0603" H 3700 5700 60  0001 C CNN
 F 3 "" H 3700 5700 60  0000 C CNN
+F 4 "Panasonic Electronic Components" H 0   0   50  0001 C CNN "Mfg"
+F 5 "EXB-38V101JV" H 0   0   50  0001 C CNN "PN"
 	4    3700 5700
 	0    1    1    0
@@
 F 2 "pkl_dipol:R_Array_Concave_4x0603" H 3700 5900 60  0001 C CNN
 F 3 "" H 3700 5900 60  0000 C CNN
+F 4 "Panasonic Electronic Components" H 0   0   50  0001 C CNN "Mfg"
+F 5 "EXB-38V101JV" H 0   0   50  0001 C CNN "PN"
 	1    3700 5900
 	0    1    1    0
@@
 F 2 "pkl_dipol:R_Array_Concave_4x0603" H 3700 6100 60  0001 C CNN
 F 3 "" H 3700 6100 60  0000 C CNN
+F 4 "Panasonic Electronic Components" H 0   0   50  0001 C CNN "Mfg"
+F 5 "EXB-38V101JV" H 0   0   50  0001 C CNN "PN"
 	2    3700 6100
 	0    1    1    0
@@
 F 2 "pkl_dipol:R_Array_Concave_4x0603" H 3700 6950 60  0001 C CNN
 F 3 "" H 3700 6950 60  0000 C CNN
+F 4 "Panasonic Electronic Components" H 0   0   50  0001 C CNN "Mfg"
+F 5 "EXB-38V101JV" H 0   0   50  0001 C CNN "PN"
 	3    3700 6950
 	0    1    1    0
@@
 F 2 "gkl_conn:DF12(3.0)-10DP-0.5V(86)" H 8300 3800 50  0001 C CNN
 F 3 "~" H 8300 3800 50  0001 C CNN
+F 4 "Hirose Electric Co Ltd" H 0   0   50  0001 C CNN "Mfg"
+F 5 "DF12(3.0)-10DP-0.5V(86)" H 0   0   50  0001 C CNN "PN"
 	1    8300 3800
 	-1   0    0    -1
@@
 F 2 "pkl_dipol:R_Array_Concave_4x0603" H 7500 3500 60  0001 C CNN
 F 3 "" H 7500 3500 60  0000 C CNN
+F 4 "Panasonic Electronic Components" H 0   0   50  0001 C CNN "Mfg"
+F 5 "EXB-38V101JV" H 0   0   50  0001 C CNN "PN"
 	2    7500 3500
 	0    1    1    0
@@
 F 2 "pkl_dipol:R_Array_Concave_4x0603" H 7500 3700 60  0001 C CNN
 F 3 "" H 7500 3700 60  0000 C CNN
+F 4 "Panasonic Electronic Components" H 0   0   50  0001 C CNN "Mfg"
+F 5 "EXB-38V101JV" H 0   0   50  0001 C CNN "PN"
 	3    7500 3700
 	0    1    1    0
@@
 F 2 "pkl_dipol:R_Array_Concave_4x0603" H 7500 3900 60  0001 C CNN
 F 3 "" H 7500 3900 60  0000 C CNN
+F 4 "Panasonic Electronic Components" H 0   0   50  0001 C CNN "Mfg"
+F 5 "EXB-38V101JV" H 0   0   50  0001 C CNN "PN"
 	4    7500 3900
 	0    1    1    0
@@
 F 2 "pkl_dipol:L_0402" V 9630 2300 50  0001 C CNN
 F 3 "~" H 9700 2300 50  0001 C CNN
+F 4 "Murata Electronics North America" H 0   0   50  0001 C CNN "Mfg"
+F 5 "BLM15AX102SN1D" H 0   0   50  0001 C CNN "PN"
 	1    9700 2300
 	0    1    1    0
@@
 F 2 "pkl_dipol:C_0603" H 9000 3900 50  0001 C CNN
 F 3 "~" H 9000 3900 50  0001 C CNN
+F 4 "Samsung Electro-Mechanics" H 0   0   50  0001 C CNN "Mfg"
+F 5 "CL10A106MQ8NNNC" H 0   0   50  0001 C CNN "PN"
 	1    9000 3900
 	1    0    0    -1
@@
 F 2 "pkl_dipol:L_0402" V 3780 1600 50  0001 C CNN
 F 3 "~" H 3850 1600 50  0001 C CNN
+F 4 "Murata Electronics North America" H 0   0   50  0001 C CNN "Mfg"
+F 5 "BLM15AX102SN1D" H 0   0   50  0001 C CNN "PN"
 	1    3850 1600
 	0    1    1    0
@@
 F 2 "pkl_dipol:C_0402" H 4500 1850 50  0001 C CNN
 F 3 "~" H 4500 1850 50  0001 C CNN
+F 4 "Yageo" H 0   0   50  0001 C CNN "Mfg"
+F 5 "CC0402KRX5R6BB105" H 0   0   50  0001 C CNN "PN"
 	1    4500 1850
 	1    0    0    -1
@@
 F 2 "pkl_dipol:C_0402" H 4900 1850 50  0001 C CNN
 F 3 "~" H 4900 1850 50  0001 C CNN
+F 4 "Yageo" H 0   0   50  0001 C CNN "Mfg"
+F 5 "CC0402KRX5R6BB104" H 0   0   50  0001 C CNN "PN"
 	1    4900 1850
 	1    0    0    -1
@@
 F 2 "pkl_dipol:C_0402" H 9400 3900 50  0001 C CNN
 F 3 "~" H 9400 3900 50  0001 C CNN
+F 4 "Yageo" H 0   0   50  0001 C CNN "Mfg"
+F 5 "CC0402KRX5R6BB104" H 0   0   50  0001 C CNN "PN"
 	1    9400 3900
 	1    0    0    -1
@@
 F 2 "pkl_dipol:C_0402" H 9800 3900 50  0001 C CNN
 F 3 "~" H 9800 3900 50  0001 C CNN
+F 4 "Yageo" H 0   0   50  0001 C CNN "Mfg"
+F 5 "CC0402KRX5R6BB104" H 0   0   50  0001 C CNN "PN"
 	1    9800 3900
 	1    0    0    -1
@@
 F 2 "" H 4300 7150 50  0001 C CNN
 F 3 "" H 4300 7150 50  0001 C CNN
+F 4 "Panasonic Electronic Components" H 0   0   50  0001 C CNN "Mfg"
+F 5 "EVQ-P1D05M" H 0   0   50  0001 C CNN "PN"
 	1    4300 6950
 	1    0    0    -1
@@
 F 2 "pkl_dipol:C_0402" H 3350 7200 50  0001 C CNN
 F 3 "~" H 3350 7200 50  0001 C CNN
+F 4 "Yageo" H 0   0   50  0001 C CNN "Mfg"
+F 5 "CC0402KRX5R6BB104" H 0   0   50  0001 C CNN "PN"
 	1    3350 7200
 	1    0    0    -1

Commit message: Update LED resistors to 330R to limit max current to 5mA
Parts:
- R2, R3, R4: value 100R -> 330R; PN EXB-38V101JV -> EXB-38V331JV
Changed lines of the file:
@@
 P 3700 4800
 F 0 "R3" V 3600 4650 50  0000 C CNN
-F 1 "100R" V 3600 4950 50  0000 C CNN
+F 1 "330R" V 3600 4950 50  0000 C CNN
 F 2 "pkl_dipol:R_Array_Concave_4x0603" H 3700 4800 60  0001 C CNN
 F 3 "" H 3700 4800 60  0000 C CNN
 F 4 "Panasonic Electronic Components" H 0   0   50  0001 C CNN "Mfg"
-F 5 "EXB-38V101JV" H 0   0   50  0001 C CNN "PN"
+F 5 "EXB-38V331JV" H 0   0   50  0001 C CNN "PN"
 	1    3700 4800
 	0    1    1    0
@@
 P 3700 5000
 F 0 "R3" V 3600 4850 50  0000 C CNN
-F 1 "100R" V 3600 5150 50  0000 C CNN
+F 1 "330R" V 3600 5150 50  0000 C CNN
 F 2 "pkl_dipol:R_Array_Concave_4x0603" H 3700 5000 60  0001 C CNN
 F 3 "" H 3700 5000 60  0000 C CNN
 F 4 "Panasonic Electronic Components" H 0   0   50  0001 C CNN "Mfg"
-F 5 "EXB-38V101JV" H 0   0   50  0001 C CNN "PN"
+F 5 "EXB-38V331JV" H 0   0   50  0001 C CNN "PN"
 	2    3700 5000
 	0    1    1    0
@@
 P 3700 5200
 F 0 "R3" V 3600 5050 50  0000 C CNN
-F 1 "100R" V 3600 5350 50  0000 C CNN
+F 1 "330R" V 3600 5350 50  0000 C CNN
 F 2 "pkl_dipol:R_Array_Concave_4x0603" H 3700 5200 60  0001 C CNN
 F 3 "" H 3700 5200 60  0000 C CNN
 F 4 "Panasonic Electronic Components" H 0   0   50  0001 C CNN "Mfg"
-F 5 "EXB-38V101JV" H 0   0   50  0001 C CNN "PN"
+F 5 "EXB-38V331JV" H 0   0   50  0001 C CNN "PN"
 	3    3700 5200
 	0    1    1    0
@@
 P 3700 5700
 F 0 "R3" V 3600 5550 50  0000 C CNN
-F 1 "100R" V 3600 5850 50  0000 C CNN
+F 1 "330R" V 3600 5850 50  0000 C CNN
 F 2 "pkl_dipol:R_Array_Concave_4x0603" H 3700 5700 60  0001 C CNN
 F 3 "" H 3700 5700 60  0000 C CNN
 F 4 "Panasonic Electronic Components" H 0   0   50  0001 C CNN "Mfg"
-F 5 "EXB-38V101JV" H 0   0   50  0001 C CNN "PN"
+F 5 "EXB-38V331JV" H 0   0   50  0001 C CNN "PN"
 	4    3700 5700
 	0    1    1    0
@@
 P 3700 5900
 F 0 "R2" V 3600 5750 50  0000 C CNN
-F 1 "100R" V 3600 6050 50  0000 C CNN
+F 1 "330R" V 3600 6050 50  0000 C CNN
 F 2 "pkl_dipol:R_Array_Concave_4x0603" H 3700 5900 60  0001 C CNN
 F 3 "" H 3700 5900 60  0000 C CNN
 F 4 "Panasonic Electronic Components" H 0   0   50  0001 C CNN "Mfg"
-F 5 "EXB-38V101JV" H 0   0   50  0001 C CNN "PN"
+F 5 "EXB-38V331JV" H 0   0   50  0001 C CNN "PN"
 	1    3700 5900
 	0    1    1    0
@@
 P 3700 6100
 F 0 "R2" V 3600 5950 50  0000 C CNN
-F 1 "100R" V 3600 6250 50  0000 C CNN
+F 1 "330R" V 3600 6250 50  0000 C CNN
 F 2 "pkl_dipol:R_Array_Concave_4x0603" H 3700 6100 60  0001 C CNN
 F 3 "" H 3700 6100 60  0000 C CNN
 F 4 "Panasonic Electronic Components" H 0   0   50  0001 C CNN "Mfg"
-F 5 "EXB-38V101JV" H 0   0   50  0001 C CNN "PN"
+F 5 "EXB-38V331JV" H 0   0   50  0001 C CNN "PN"
 	2    3700 6100
 	0    1    1    0
@@
 P 3700 6950
 F 0 "R2" V 3800 6800 50  0000 C CNN
-F 1 "100R" V 3750 7100 50  0000 C CNN
+F 1 "330R" V 3750 7100 50  0000 C CNN
 F 2 "pkl_dipol:R_Array_Concave_4x0603" H 3700 6950 60  0001 C CNN
 F 3 "" H 3700 6950 60  0000 C CNN
 F 4 "Panasonic Electronic Components" H 0   0   50  0001 C CNN "Mfg"
-F 5 "EXB-38V101JV" H 0   0   50  0001 C CNN "PN"
+F 5 "EXB-38V331JV" H 0   0   50  0001 C CNN "PN"
 	3    3700 6950
 	0    1    1    0
@@
 P 7500 3500
 F 0 "R4" V 7400 3350 50  0000 C CNN
-F 1 "100R" V 7400 3650 50  0000 C CNN
+F 1 "330R" V 7400 3650 50  0000 C CNN
 F 2 "pkl_dipol:R_Array_Concave_4x0603" H 7500 3500 60  0001 C CNN
 F 3 "" H 7500 3500 60  0000 C CNN
 F 4 "Panasonic Electronic Components" H 0   0   50  0001 C CNN "Mfg"
-F 5 "EXB-38V101JV" H 0   0   50  0001 C CNN "PN"
+F 5 "EXB-38V331JV" H 0   0   50  0001 C CNN "PN"
 	2    7500 3500
 	0    1    1    0
@@
 P 7500 3700
 F 0 "R4" V 7400 3550 50  0000 C CNN
-F 1 "100R" V 7400 3850 50  0000 C CNN
+F 1 "330R" V 7400 3850 50  0000 C CNN
 F 2 "pkl_dipol:R_Array_Concave_4x0603" H 7500 3700 60  0001 C CNN
 F 3 "" H 7500 3700 60  0000 C CNN
 F 4 "Panasonic Electronic Components" H 0   0   50  0001 C CNN "Mfg"
-F 5 "EXB-38V101JV" H 0   0   50  0001 C CNN "PN"
+F 5 "EXB-38V331JV" H 0   0   50  0001 C CNN "PN"
 	3    7500 3700
 	0    1    1    0
@@
 P 7500 3900
 F 0 "R4" V 7400 3750 50  0000 C CNN
-F 1 "100R" V 7400 4050 50  0000 C CNN
+F 1 "330R" V 7400 4050 50  0000 C CNN
 F 2 "pkl_dipol:R_Array_Concave_4x0603" H 7500 3900 60  0001 C CNN
 F 3 "" H 7500 3900 60  0000 C CNN
 F 4 "Panasonic Electronic Components" H 0   0   50  0001 C CNN "Mfg"
-F 5 "EXB-38V101JV" H 0   0   50  0001 C CNN "PN"
+F 5 "EXB-38V331JV" H 0   0   50  0001 C CNN "PN"
 	4    7500 3900
 	0    1    1    0
