File: hardware/v0.1a/gpsLoggerLoRa.kicad_pcb (KiCad board)
At the start: 4 copper layers, 40.9 x 72.7 mm, 120 parts, among them J1 USB_C_Receptacle, J2 JST GH, J3 DF12 - 10P, J4 CTX TAG Connect, Q1 FG6943010R, SW1 SW_Push, U1 SKY13373, U2 MCP73832, U3 NCP167, U4 SKY13373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

Commit message: Fixed a DRC error in the GPS PCB. Small layout change to include a logo/product name on the PCB. Created a prototype 'panel' with both PCB attached for production.
Parts:
- added G***: LOGO, LOGO, F.Cu at (155.1, 91.3)
- moved G*** 27.5 mm to (158.8, 94.0), turned to 90 degrees
- moved G*** 25.1 mm to (158.8, 90.5), turned to 90 degrees
- moved C16 1.17 mm to (158.8, 97.3), turned to 90 degrees
Routing:
- net Net-(R2-Pad5): track 26.9 -> 33.2 mm
- net /USB/VBAT: track 41.6 -> 45.2 mm, vias 5 -> 6
- net GND: track 122.8 -> 121.9 mm, vias 212 -> 213
