File: hardware/gps-v0.1a/gpsDaughterBoard.sch (KiCad schematic (older format))
At the start: 8 parts, among them J1 JST DF12 10P, U1 NEO_M8, U2 BGU7007

Commit message: First Pass routing GPS board
Connections:
- net labels added: PPS, RX, TX
Other:
- note added: "<"
- note added: ">"
Changed lines of the file:
@@
 EESchema Schematic File Version 4
-LIBS:gpsLoggerLoRa-cache
+LIBS:gpsDaughterBoard-cache
 EELAYER 26 0
 EELAYER END
@@
 	3250 2800 3850 2800
 Wire Wire Line
-	4100 4400 3300 4400
-Wire Wire Line
-	3300 4400 3300 3850
-Wire Wire Line
-	3300 3850 2950 3850
-Wire Wire Line
-	2950 3750 3400 3750
-Wire Wire Line
-	3400 3750 3400 4300
-Wire Wire Line
-	3400 4300 4100 4300
-Wire Wire Line
 	5600 4500 5800 4500
 Wire Wire Line
 	5800 4500 5800 5000
-Wire Wire Line
-	5800 5000 3500 5000
-Wire Wire Line
-	3500 5000 3500 3650
-Wire Wire Line
-	3500 3650 2950 3650
 Wire Wire Line
 	4100 4700 3950 4700
@@
 Wire Wire Line
 	9000 3600 9000 3200
+Wire Wire Line
+	2950 3650 3650 3650
+Wire Wire Line
+	3650 3650 3650 4400
+Wire Wire Line
+	3650 4400 4100 4400
+Wire Wire Line
+	4100 4300 3550 4300
+Wire Wire Line
+	3550 4300 3550 3750
+Wire Wire Line
+	3550 3750 2950 3750
+Wire Wire Line
+	2950 3850 3450 3850
+Wire Wire Line
+	3450 3850 3450 5000
+Wire Wire Line
+	3450 5000 5800 5000
+Text Label 3150 3650 0    60   ~ 0
+TX
+Text Label 3150 3750 0    60   ~ 0
+RX
+Text Label 3150 3850 0    60   ~ 0
+PPS
+Text Notes 3300 3750 0    60   ~ 0
+<
+Text Notes 3300 3650 0    60   ~ 0
+>
 $EndSCHEMATC

Commit message: Added BOM part numbers to GPS PCB.
Parts:
- added C4: 1nF, pkl_dipol:C_0402, symbol device:C
- added FLT2: SF1186G, gkl_housings_son:SAW-5, symbol gkl_rf:SF1186G
- added L1: 5.6nH, pkl_dipol:L_0402, symbol device:L
- C1: footprint (none) -> pkl_dipol:C_0402; Mfg (none) -> Yageo; PN (none) -> CC0402KRX7R8BB103
- C2, C3: footprint (none) -> pkl_dipol:C_0402; Mfg (none) -> Yageo; PN (none) -> CC0402KRX5R6BB104
- FLT1: Mfg (none) -> Qualcomm (RF360 - A Qualcomm & TDK Joint Venture); PN (none) -> B39162B8828P810
- J1: footprint (none) -> gkl_conn:DF12(3.0)-10DS-0.5V(86); Mfg (none) -> Hirose Electric Co Ltd; PN (none) -> DF12(3.0)-10DS-0.5V(86)
- U1: Mfg (none) -> Ublox; PN (none) -> NEO series
- U2: Mfg (none) -> NXP USA Inc.; PN (none) -> BGU7007,115
Connections:
- wire segments 50 -> 65
Changed lines of the file:
@@
 F 2 "gkl_ublox:NEO-M8" H 4850 4484 60  0000 C CNN
 F 3 "" H 4850 3875 60  0000 C CNN
+F 4 "Ublox" H 0   0   50  0001 C CNN "Mfg"
+F 5 "NEO series" H 0   0   50  0001 C CNN "PN"
 	1    4850 3900
 	1    0    0    -1
@@
 F 0 "C1" H 2600 3150 50  0000 L CNN
 F 1 "10nF" H 2600 2950 50  0000 L CNN
-F 2 "" H 2588 2900 50  0001 C CNN
+F 2 "pkl_dipol:C_0402" H 2588 2900 50  0001 C CNN
 F 3 "~" H 2550 3050 50  0001 C CNN
+F 4 "Yageo" H 0   0   50  0001 C CNN "Mfg"
+F 5 "CC0402KRX7R8BB103" H 0   0   50  0001 C CNN "PN"
 	1    2550 3050
 	1    0    0    -1
@@
 L gkl_rf:BGU7007 U2
 U 1 1 5C281203
-P 7000 3600
-F 0 "U2" H 6800 3450 60  0000 R CNN
-F 1 "BGU7007" H 6800 3750 60  0000 R CNN
-F 2 "gkl_housings_son:XSON6" H 7000 3600 60  0001 C CNN
-F 3 "" H 7000 3600 60  0000 C CNN
-	1    7000 3600
+P 7250 3600
+F 0 "U2" H 7050 3450 60  0000 R CNN
+F 1 "BGU7007" H 7050 3750 60  0000 R CNN
+F 2 "gkl_housings_son:XSON6" H 7250 3600 60  0001 C CNN
+F 3 "" H 7250 3600 60  0000 C CNN
+F 4 "NXP USA Inc." H 250 0   50  0001 C CNN "Mfg"
+F 5 "BGU7007,115" H 250 0   50  0001 C CNN "PN"
+	1    7250 3600
 	-1   0    0    1
 $EndComp
@@
 L gkl_rf:SF1186G FLT1
 U 1 1 5C281252
-P 8100 3600
-F 0 "FLT1" H 8100 3260 60  0000 C CNN
-F 1 "SF1186G" H 8100 3366 60  0000 C CNN
-F 2 "gkl_housings_son:SAW-5" H 8100 3366 60  0001 C CNN
-F 3 "" H 7700 4050 60  0000 C CNN
-	1    8100 3600
+P 6350 3600
+F 0 "FLT1" H 6350 3260 60  0000 C CNN
+F 1 "SF1186G" H 6350 3366 60  0000 C CNN
+F 2 "gkl_housings_son:SAW-5" H 6350 3366 60  0001 C CNN
+F 3 "" H 5950 4050 60  0000 C CNN
+F 4 "B39162B8828P810" H -1750 0   50  0001 C CNN "PN"
+F 5 "Qualcomm (RF360 - A Qualcomm & TDK Joint Venture)" H -1750 0   50  0001 C CNN "Mfg"
+	1    6350 3600
 	-1   0    0    1
 $EndComp
@@
 F 0 "J1" H 2700 4267 50  0000 C CNN
 F 1 "JST DF12 10P" H 2700 4176 50  0000 C CNN
-F 2 "" H 2650 3850 50  0001 C CNN
+F 2 "gkl_conn:DF12(3.0)-10DS-0.5V(86)" H 2650 3850 50  0001 C CNN
 F 3 "~" H 2650 3850 50  0001 C CNN
+F 4 "Hirose Electric Co Ltd" H 0   0   50  0001 C CNN "Mfg"
+F 5 "DF12(3.0)-10DS-0.5V(86)" H 0   0   50  0001 C CNN "PN"
 	1    2650 3850
 	1    0    0    -1
@@
 F 0 "C2" H 2950 3150 50  0000 L CNN
 F 1 "100nF" H 2950 2950 50  0000 L CNN
-F 2 "" H 2938 2900 50  0001 C CNN
+F 2 "pkl_dipol:C_0402" H 2938 2900 50  0001 C CNN
 F 3 "~" H 2900 3050 50  0001 C CNN
+F 4 "Yageo" H 0   0   50  0001 C CNN "Mfg"
+F 5 "CC0402KRX5R6BB104" H 0   0   50  0001 C CNN "PN"
 	1    2900 3050
 	1    0    0    -1
@@
 F 0 "C3" H 3300 3150 50  0000 L CNN
 F 1 "100nF" H 3300 2950 50  0000 L CNN
-F 2 "" H 3288 2900 50  0001 C CNN
+F 2 "pkl_dipol:C_0402" H 3288 2900 50  0001 C CNN
 F 3 "~" H 3250 3050 50  0001 C CNN
+F 4 "Yageo" H 0   0   50  0001 C CNN "Mfg"
+F 5 "CC0402KRX5R6BB104" H 0   0   50  0001 C CNN "PN"
 	1    3250 3050
 	1    0    0    -1
@@
 	5900 3700 5900 4000
 Wire Wire Line
-	5600 3600 6750 3600
+	6650 3600 7000 3600
 $Comp
 L power:GND #PWR0106
@@
 $EndComp
 Wire Wire Line
-	7800 3600 7250 3600
-Wire Wire Line
-	8400 3600 9000 3600
+	8900 3600 9000 3600
 Wire Wire Line
 	9000 3600 9000 3200
@@
 Text Notes 3300 3650 0    60   ~ 0
 >
+Wire Wire Line
+	7200 3400 7200 3150
+Wire Wire Line
+	7300 3400 7300 3150
+Wire Wire Line
+	7300 3150 7200 3150
+Connection ~ 7200 3150
+Wire Wire Line
+	7200 3800 7200 3900
+Wire Wire Line
+	7200 3900 7300 3900
+Wire Wire Line
+	7300 3800 7300 3900
+Connection ~ 7300 3900
+Wire Wire Line
+	7300 3900 7300 4050
+$Comp
+L power:GND #PWR0108
+U 1 1 5C27B39E
+P 7300 4050
+F 0 "#PWR0108" H 7300 3800 50  0001 C CNN
+F 1 "GND" H 7303 3924 50  0000 C CNN
+F 2 "" H 7200 3700 50  0001 C CNN
+F 3 "" H 7300 4050 50  0001 C CNN
+	1    7300 4050
+	1    0    0    -1
+$EndComp
+Wire Wire Line
+	6050 3600 5600 3600
+Wire Wire Line
+	5600 3800 5700 3800
+Wire Wire Line
+	5700 3800 5700 3150
+Wire Wire Line
+	5700 3150 7200 3150
+$Comp
+L gkl_rf:SF1186G FLT2
+U 1 1 5C28347F
+P 8600 3600
+F 0 "FLT2" H 8600 3260 60  0000 C CNN
+F 1 "SF1186G" H 8600 3366 60  0000 C CNN
+F 2 "gkl_housings_son:SAW-5" H 8600 3366 60  0001 C CNN
+F 3 "" H 8200 4050 60  0000 C CNN
+F 4 "B39162B8828P810" H 500 0   50  0001 C CNN "PN"
+F 5 "Qualcomm (RF360 - A Qualcomm & TDK Joint Venture)" H 500 0   50  0001 C CNN "Mfg"
+	1    8600 3600
+	-1   0    0    1
+$EndComp
+$Comp
+L device:L L1
+U 1 1 5C285083
+P 7950 3600
+F 0 "L1" V 8140 3600 50  0000 C CNN
+F 1 "5.6nH" V 8049 3600 50  0000 C CNN
+F 2 "pkl_dipol:L_0402" H 7950 3600 50  0001 C CNN
+F 3 "~" H 7950 3600 50  0001 C CNN
+	1    7950 3600
+	0    -1   -1   0
+$EndComp
+Wire Wire Line
+	8300 3600 8100 3600
+Wire Wire Line
+	7800 3600 7500 3600
+$Comp
+L device:C C4
+U 1 1 5C286D90
+P 7650 3000
+F 0 "C4" H 7700 3100 50  0000 L CNN
+F 1 "1nF" H 7700 2900 50  0000 L CNN
+F 2 "pkl_dipol:C_0402" H 7688 2850 50  0001 C CNN
+F 3 "~" H 7650 3000 50  0001 C CNN
+F 4 "Yageo" H 5100 -50 50  0001 C CNN "Mfg"
+F 5 "CC0402KRX7R8BB103" H 5100 -50 50  0001 C CNN "PN"
+	1    7650 3000
+	1    0    0    -1
+$EndComp
+Wire Wire Line
+	7300 3150 7300 2750
+Wire Wire Line
+	7300 2750 7650 2750
+Wire Wire Line
+	7650 2750 7650 2850
+Connection ~ 7300 3150
+$Comp
+L power:GND #PWR0109
+U 1 1 5C287D99
+P 7650 3150
+F 0 "#PWR0109" H 7650 2900 50  0001 C CNN
+F 1 "GND" H 7653 3024 50  0000 C CNN
+F 2 "" H 7550 2800 50  0001 C CNN
+F 3 "" H 7650 3150 50  0001 C CNN
+	1    7650 3150
+	1    0    0    -1
+$EndComp
 $EndSCHEMATC

Commit message: Updated GPS pcb with impoved RF path, and potetially easier to solder filters. Added USB connector to GPS pcb for debugging ublox.
Parts:
- added J2: USB_OTG, symbol conn:USB_OTG
Connections:
- net labels added: DATA_N, DATA_P
- wire segments 65 -> 78
